File: double_145MHz_BPF.kicad_sch (KiCad schematic)
At the start: 5 parts, among them J1 Conn_01x02_Socket, J2 Conn_01x02_Socket, J3 Conn_01x01_Socket, U1 SXBP-140, U2 SXBP-140

Commit message: new gerber, vna analyze, test setup pictures
Connections:
- net at J1.1 (Pin_1): now also U2.8 (OUT); no longer U2.1 (IN)
- net at U1.8 (OUT): now also U2.1 (IN); no longer U2.8 (OUT)
Changed lines of the file:
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@@
+	(wire
+		(pts
+			(xy 99.314 48.26) (xy 100.076 48.26)
+		)
+		(stroke
+			(width 0)
+			(type default)
+		)
+	)
 	(wire
 		(pts
@@
 	(wire
 		(pts
-			(xy 93.726 58.42) (xy 93.726 59.944)
-		)
-		(stroke
-			(width 0)
-			(type default)
-		)
-	)
-	(wire
-		(pts
 			(xy 55.118 50.8) (xy 55.118 52.324)
 		)
@@
 	(wire
 		(pts
+			(xy 84.074 58.42) (xy 84.074 59.944)
+		)
+		(stroke
+			(width 0)
+			(type default)
+		)
+	)
+	(wire
+		(pts
 			(xy 69.596 58.674) (xy 69.596 60.198)
 		)
@@
 	(wire
 		(pts
-			(xy 76.962 48.26) (xy 78.486 48.26)
-		)
-		(stroke
-			(width 0)
-			(type default)
-		)
-	)
-	(wire
-		(pts
-			(xy 98.806 48.26) (xy 100.076 48.26)
+			(xy 76.962 48.26) (xy 78.994 48.26)
 		)
 		(stroke
@@
 	)
 	(symbol
-		(lib_id "power:GND")
-		(at 93.726 59.944 0)
-		(unit 1)
-		(exclude_from_sim no)
-		(in_bom yes)
-		(on_board yes)
-		(dnp no)
-		(fields_autoplaced yes)
-		(property "Reference" "#PWR05"
-			(at 93.726 66.294 0)
-			(effects
-				(font
-					(size 1.27 1.27)
-				)
-				(hide yes)
-			)
-		)
-		(property "Value" "GND"
-			(at 93.726 64.0771 0)
-			(effects
-				(font
-					(size 1.27 1.27)
-				)
-			)
-		)
-		(property "Footprint" ""
-			(at 93.726 59.944 0)
-			(effects
-				(font
-					(size 1.27 1.27)
-				)
-				(hide yes)
-			)
-		)
-		(property "Datasheet" ""
-			(at 93.726 59.944 0)
-			(effects
-				(font
-					(size 1.27 1.27)
-				)
-				(hide yes)
-			)
-		)
-		(property "Description" "Power symbol creates a global label with name \"GND\" , ground"
-			(at 93.726 59.944 0)
-			(effects
-				(font
-					(size 1.27 1.27)
-				)
-				(hide yes)
-			)
-		)
-		(pin "1"
-		)
-		(instances
-			(project "145MHz_BPF"
-				(path "/400861fc-cbc3-4ec9-a9e3-afcce8493da3"
-					(reference "#PWR05")
-					(unit 1)
-				)
-			)
-		)
-	)
-	(symbol
 		(lib_id "Connector:Conn_01x02_Socket")
 		(at 50.038 48.26 0)
@@
 	)
 	(symbol
-		(lib_id "RF_Filter:SXBP-140")
-		(at 88.646 48.26 0)
-		(mirror y)
-		(unit 1)
-		(exclude_from_sim no)
-		(in_bom yes)
-		(on_board yes)
-		(dnp no)
-		(property "Reference" "U2"
-			(at 88.646 37.7655 0)
-			(effects
-				(font
-					(size 1.27 1.27)
-				)
-			)
-		)
-		(property "Value" "SXBP-140"
-			(at 88.646 40.1898 0)
-			(effects
-				(font
-					(size 1.27 1.27)
-				)
-			)
-		)
-		(property "Footprint" "RF_Mini-Circuits:Mini-Circuits_HF1139_LandPatternPL-230"
-			(at 88.646 59.69 0)
-			(effects
-				(font
-					(size 1.27 1.27)
-				)
-				(hide yes)
-			)
-		)
-		(property "Datasheet" "https://www.minicircuits.com/pdfs/SXBP-140+.pdf"
-			(at 88.646 38.1 0)
-			(effects
-				(font
-					(size 1.27 1.27)
-				)
-				(hide yes)
-			)
-		)
-		(property "Description" "Bandpass Filter, 130 to 150 MHz, 50 Ohm, Mini-Circuits HF1139"
-			(at 88.646 48.26 0)
-			(effects
-				(font
-					(size 1.27 1.27)
-				)
-				(hide yes)
-			)
-		)
-		(pin "8"
-		)
-		(pin "5"
-		)
-		(pin "4"
-		)
-		(pin "6"
-		)
-		(pin "2"
-		)
-		(pin "1"
-		)
-		(pin "7"
-		)
-		(pin "3"
-		)
-		(instances
-			(project "145MHz_BPF"
-				(path "/400861fc-cbc3-4ec9-a9e3-afcce8493da3"
-					(reference "U2")
+		(lib_id "power:GND")
+		(at 84.074 59.944 0)
+		(unit 1)
+		(exclude_from_sim no)
+		(in_bom yes)
+		(on_board yes)
+		(dnp no)
+		(fields_autoplaced yes)
+		(property "Reference" "#PWR05"
+			(at 84.074 66.294 0)
+			(effects
+				(font
+					(size 1.27 1.27)
+				)
+				(hide yes)
+			)
+		)
+		(property "Value" "GND"
+			(at 84.074 64.0771 0)
+			(effects
+				(font
+					(size 1.27 1.27)
+				)
+			)
+		)
+		(property "Footprint" ""
+			(at 84.074 59.944 0)
+			(effects
+				(font
+					(size 1.27 1.27)
+				)
+				(hide yes)
+			)
+		)
+		(property "Datasheet" ""
+			(at 84.074 59.944 0)
+			(effects
+				(font
+					(size 1.27 1.27)
+				)
+				(hide yes)
+			)
+		)
+		(property "Description" "Power symbol creates a global label with name \"GND\" , ground"
+			(at 84.074 59.944 0)
+			(effects
+				(font
+					(size 1.27 1.27)
+				)
+				(hide yes)
+			)
+		)
+		(pin "1"
+		)
+		(instances
+			(project "double_145MHz_BPF"
+				(path "/400861fc-cbc3-4ec9-a9e3-afcce8493da3"
+					(reference "#PWR05")
 					(unit 1)
 				)
@@
 					(unit 1)
 				)
+			)
+		)
+	)
+	(symbol
+		(lib_id "RF_Filter:SXBP-140")
+		(at 89.154 48.26 0)
+		(unit 1)
+		(exclude_from_sim no)
+		(in_bom yes)
+		(on_board yes)
+		(dnp no)
+		(fields_autoplaced yes)
+		(property "Reference" "U2"
+			(at 89.154 37.7655 0)
+			(effects
+				(font
+					(size 1.27 1.27)
+				)
+			)
+		)
+		(property "Value" "SXBP-140"
+			(at 89.154 40.1898 0)
+			(effects
+				(font
+					(size 1.27 1.27)
+				)
+			)
+		)
+		(property "Footprint" "RF_Mini-Circuits:Mini-Circuits_HF1139_LandPatternPL-230"
+			(at 89.154 59.69 0)
+			(effects
+				(font
+					(size 1.27 1.27)
+				)
+				(hide yes)
+			)
+		)
+		(property "Datasheet" "https://www.minicircuits.com/pdfs/SXBP-140+.pdf"
+			(at 89.154 38.1 0)
+			(effects
+				(font
+					(size 1.27 1.27)
+				)
+				(hide yes)
+			)
+		)
+		(property "Description" "Bandpass Filter, 130 to 150 MHz, 50 Ohm, Mini-Circuits HF1139"
+			(at 89.154 48.26 0)
+			(effects
+				(font
+					(size 1.27 1.27)
+				)
+				(hide yes)
+			)
+		)
+		(pin "8"
+		)
+		(pin "5"
+		)
+		(pin "4"
+		)
+		(pin "6"
+		)
+		(pin "2"
+		)
+		(pin "1"
+		)
+		(pin "7"
+		)
+		(pin "3"
+		)
+		(instances
+			(project "double_145MHz_BPF"
+				(path "/400861fc-cbc3-4ec9-a9e3-afcce8493da3"
+					(reference "U2")
+					(unit 1)
+				)
